File: pcb/gingham.sch (KiCad schematic (older format))
At the start: 171 parts, among them J1 USB4085-GF-A_REVA, J2 ISP, J3 I2C, SW1 SW_Push, SW10 SW_Push, SW11 SW_Push, SW12 SW_Push, SW13 SW_Push, SW14 SW_Push, SW15 SW_Push, SW16 SW_Push, SW17 SW_Push, SW18 SW_Push, SW19 SW_Push, SW2 SW_Push, SW20 SW_Push, SW21 SW_Push, SW22 SW_Push, SW23 SW_Push, SW24 SW_Push, SW25 SW_Push, SW26 SW_Push, SW27 SW_Push, SW28 SW_Push, SW29 SW_Push, SW3 SW_Push, SW30 SW_Push, SW31 SW_Push, SW32 SW_Push, SW33 SW_Push, SW34 SW_Push, SW35 SW_Push, SW36 SW_Push, SW37 SW_Push, SW38 SW_Push, SW39 SW_Push, SW4 SW_Push, SW40 SW_Push, SW41 SW_Push, SW42 SW_Push, SW43 SW_Push, SW44 SW_Push, SW45 SW_Push, SW46 SW_Push, SW47 SW_Push, SW48 SW_Push, SW49 SW_Push, SW5 SW_Push, SW50 SW_Push, SW51 SW_Push, SW52 SW_Push, SW53 SW_Push, SW54 SW_Push, SW55 SW_Push, SW56 SW_Push, SW57 SW_Push, SW58 SW_Push, SW59 SW_Push, SW6 SW_Push, SW60 SW_Push, SW61 SW_Push, SW62 SW_Push, SW63 SW_Push, SW64 SW_Push, SW65 SW_Push, SW66 SW_Push, SW67 SW_Push, SW68 RESET, SW69 BOOT, SW7 SW_Push, SW70 SW_Push, SW71 SW_Push, SW8 SW_Push, SW9 SW_Push, U1 ATMEGA328-PU, U2 MCP23008-E_P, Y1 16MHz

Commit message: Update Instructions
Changed lines of the file:
@@
 U 1 1 5C16FB14
 P 2125 5525
-F 0 "U1" H 2175 6892 50  0000 C CNN
-F 1 "ATMEGA328-PU" H 2175 6801 50  0000 C CNN
+F 0 "U1" H 2825 7050 50  0000 C CNN
+F 1 "ATMEGA328-PU" H 2575 6975 50  0000 C CNN
 F 2 "Package_DIP:DIP-28_W7.62mm" H 2125 5525 50  0001 C CIN
 F 3 "http://www.atmel.com/images/atmel-8271-8-bit-avr-microcontroller-atmega48a-48pa-88a-88pa-168a-168pa-328-328p_datasheet.pdf" H 2125 5525 50  0001 C CNN
@@
 	1    0    0    -1
 $EndComp
-Wire Wire Line
-	2125 10325 2125 10375
 $Comp
 L power:GND #PWR0103
@@
 Wire Wire Line
 	4650 3375 4725 3375
-Text Notes 2675 10100 0    50   ~ 6
+Text Notes 2675 10100 0    50   ~ 10
 Address: 0x20
 $Comp
@@
 Wire Wire Line
 	2300 1475 2300 1625
+Wire Wire Line
+	2125 10325 2125 10375
+$Comp
+L power:PWR_FLAG #FLG0101
+U 1 1 5F1CDB56
+P 1825 2225
+F 0 "#FLG0101" H 1825 2275 25  0001 C CNN
+F 1 "PWR_FLAG" H 1825 2354 25  0000 C CNN
+F 2 "" H 1825 2225 50  0000 C CNN
+F 3 "" H 1825 2225 50  0000 C CNN
+	1    1825 2225
+	1    0    0    -1
+$EndComp
+Wire Wire Line
+	1750 2225 1825 2225
 $EndSCHEMATC
