File: pcb/gingham.kicad_pcb (KiCad board)
At the start: 2 copper layers, 285.8 x 123.8 mm, 173 parts, among them J1 USB4085-GF-A_REVA, J2 ISP, J3 I2C, SW1 SW_Push, SW10 SW_Push, SW11 SW_Push, SW12 SW_Push, SW13 SW_Push, SW14 SW_Push, SW15 SW_Push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

Commit message: Update Instructions
Other:
- rule pad_to_mask_clearance: 0.2 -> 0
